File: PCM2707_DAC.brd (EAGLE design)
At the start: 49.6 x 38.1 mm, 37 parts, among them CON1 GND_CONNECTORSMD, Q1 12MHz

Commit message: Added updated files, and PDF of data
Parts:
- J1: value (none) -> USB
- OUTPUT: value (none) -> AUDIO
- SV1: value (none) -> USB-WIRE
