File: PCM2707_DAC.sch (EAGLE design)
At the start: 37 parts, among them CON1 GND_CONNECTORSMD, Q1 12MHz, U1 PCM2707C_TQFP32"

Commit message: Added updated files, and PDF of data
Parts:
- J1: value (none) -> USB
- OUTPUT: value (none) -> AUDIO
- SV1: value (none) -> USB-WIRE
Other:
- moved on the sheet: J1, OUTPUT
Changed lines of the file:
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@@
 <part name="R3" library="SparkFun-Passives" deviceset="RESISTOR" device="0805-RES" value="1.5kOhm"/>
 <part name="JACK-OUT" library="akafugu" deviceset="STEREOJACK" device=""/>
-<part name="OUTPUT" library="con-lstb" deviceset="MA03-1" device=""/>
-<part name="SV1" library="con-lstb" deviceset="MA04-1" device=""/>
+<part name="OUTPUT" library="con-lstb" deviceset="MA03-1" device="" value="AUDIO"/>
+<part name="SV1" library="con-lstb" deviceset="MA04-1" device="" value="USB-WIRE"/>
 <part name="GND11" library="SparkFun-Aesthetics" deviceset="GND" device=""/>
-<part name="J1" library="Molex-47346-0001" deviceset="47346-0001" device=""/>
+<part name="J1" library="Molex-47346-0001" deviceset="47346-0001" device="" value="USB"/>
 <part name="GND12" library="SparkFun-Aesthetics" deviceset="GND" device=""/>
 <part name="DOUT" library="con-molex" deviceset="87758-0216" device=""/>
 <part name="GND13" library="SparkFun-Aesthetics" deviceset="GND" device=""/>
+<part name="SUPPLY16" library="supply2" deviceset="AGND" device=""/>
+<part name="FRAME1" library="frames" deviceset="A3L-LOC" device=""/>
 </parts>
 <sheets>
@@
 <instance part="R3" gate="G$1" x="96.52" y="33.02" rot="R90"/>
 <instance part="JACK-OUT" gate="1" x="180.34" y="170.18"/>
-<instance part="OUTPUT" gate="G$1" x="35.56" y="195.58"/>
+<instance part="OUTPUT" gate="G$1" x="15.24" y="165.1"/>
 <instance part="SV1" gate="1" x="208.28" y="66.04" rot="R180"/>
 <instance part="GND11" gate="1" x="200.66" y="45.72"/>
-<instance part="J1" gate="G$1" x="210.82" y="7.62"/>
-<instance part="GND12" gate="1" x="200.66" y="-7.62"/>
+<instance part="J1" gate="G$1" x="17.78" y="137.16"/>
+<instance part="GND12" gate="1" x="7.62" y="121.92"/>
 <instance part="DOUT" gate="-1" x="139.7" y="55.88"/>
 <instance part="DOUT" gate="-2" x="139.7" y="50.8"/>
 <instance part="GND13" gate="1" x="121.92" y="48.26"/>
+<instance part="SUPPLY16" gate="G$1" x="27.94" y="160.02"/>
+<instance part="FRAME1" gate="G$1" x="-83.82" y="-40.64"/>
 </instances>
 <busses>
@@
 <pinref part="J1" gate="G$1" pin="5"/>
 <pinref part="GND12" gate="1" pin="GND"/>
-<wire x1="200.66" y1="-5.08" x2="200.66" y2="2.54" width="0.1524" layer="91"/>
+<wire x1="7.62" y1="124.46" x2="7.62" y2="132.08" width="0.1524" layer="91"/>
 </segment>
 <segment>
@@
 </segment>
 <segment>
-<wire x1="48.26" y1="193.04" x2="43.18" y2="193.04" width="0.1524" layer="91"/>
-<label x="40.64" y="193.04" size="1.778" layer="95"/>
+<wire x1="27.94" y1="162.56" x2="22.86" y2="162.56" width="0.1524" layer="91"/>
+<label x="20.32" y="162.56" size="1.778" layer="95"/>
 <pinref part="OUTPUT" gate="G$1" pin="1"/>
+<pinref part="SUPPLY16" gate="G$1" pin="AGND"/>
 </segment>
 </net>
@@
 <pinref part="JACK-OUT" gate="1" pin="2"/>
 <junction x="167.64" y="165.1"/>
-</segment>
-<segment>
-<wire x1="48.26" y1="195.58" x2="43.18" y2="195.58" width="0.1524" layer="91"/>
-<label x="40.64" y="195.58" size="1.778" layer="95"/>
+<label x="157.48" y="167.64" size="1.778" layer="95"/>
+</segment>
+<segment>
+<wire x1="27.94" y1="165.1" x2="22.86" y2="165.1" width="0.1524" layer="91"/>
+<label x="20.32" y="165.1" size="1.778" layer="95"/>
 <pinref part="OUTPUT" gate="G$1" pin="2"/>
 </segment>
@@
 <pinref part="JACK-OUT" gate="1" pin="5"/>
 <junction x="167.64" y="172.72"/>
-</segment>
-<segment>
-<wire x1="48.26" y1="198.12" x2="43.18" y2="198.12" width="0.1524" layer="91"/>
-<label x="40.64" y="198.12" size="1.778" layer="95"/>
+<label x="157.48" y="175.26" size="1.778" layer="95"/>
+</segment>
+<segment>
+<wire x1="27.94" y1="167.64" x2="22.86" y2="167.64" width="0.1524" layer="91"/>
+<label x="20.32" y="167.64" size="1.778" layer="95"/>
 <pinref part="OUTPUT" gate="G$1" pin="3"/>
 </segment>
@@
 <segment>
 <pinref part="J1" gate="G$1" pin="1"/>
-<wire x1="200.66" y1="12.7" x2="190.5" y2="12.7" width="0.1524" layer="91"/>
-<label x="190.5" y="12.7" size="1.778" layer="95"/>
+<wire x1="7.62" y1="142.24" x2="-2.54" y2="142.24" width="0.1524" layer="91"/>
+<label x="-2.54" y="142.24" size="1.778" layer="95"/>
 </segment>
 </net>
@@
 <segment>
 <pinref part="J1" gate="G$1" pin="2"/>
-<wire x1="200.66" y1="10.16" x2="190.5" y2="10.16" width="0.1524" layer="91"/>
-<label x="190.5" y="10.16" size="1.778" layer="95"/>
+<wire x1="7.62" y1="139.7" x2="-2.54" y2="139.7" width="0.1524" layer="91"/>
+<label x="-2.54" y="139.7" size="1.778" layer="95"/>
 </segment>
 </net>
@@
 <segment>
 <pinref part="J1" gate="G$1" pin="3"/>
-<wire x1="200.66" y1="7.62" x2="190.5" y2="7.62" width="0.1524" layer="91"/>
-<label x="190.5" y="7.62" size="1.778" layer="95"/>
+<wire x1="7.62" y1="137.16" x2="-2.54" y2="137.16" width="0.1524" layer="91"/>
+<label x="-2.54" y="137.16" size="1.778" layer="95"/>
 </segment>
 </net>
@@
 </sheet>
 </sheets>
-<errors>
-</errors>
 </schematic>
 </drawing>
