File: kicad/PCM2707_DAC.sch (KiCad schematic (older format))
At the start: 37 parts, among them CON1 GND_CONNECTORSMD, J1 USB, Q1 12MHz, U1 PCM2707C

Commit message: Converted Libs
Converted PCM2707 libs from legacy to new version
Parts:
- C1, C12, C3, C4, C5, C6, C7, C8, C9, L1, R1, R10, R11, R12, R13, R2, R3, R4, R5, R6, R7, R8, R9: footprint PCM2707_DAC:PASSIVES_0805 -> PCM2707:PASSIVES_0805
- C10, C11: footprint PCM2707_DAC:PASSIVES_PANASONIC_D -> PCM2707:PASSIVES_PANASONIC_D
- C2: footprint PCM2707_DAC:PASSIVES_PANASONIC_C -> PCM2707:PASSIVES_PANASONIC_C
- CON1: footprint PCM2707_DAC:GND_CONNECTOR -> PCM2707:GND_CONNECTOR
- DOUT1: footprint PCM2707_DAC:CON-MOLEX_87758-0216 -> PCM2707:CON-MOLEX_87758-0216
- J1: footprint PCM2707_DAC:MOLEX-47346-0001_MOLEX_47346-0001 -> PCM2707:MOLEX-47346-0001_MOLEX_47346-0001
- JACK-OUT1: footprint PCM2707_DAC:STX3100 -> PCM2707:STX3100
- JP1: footprint PCM2707_DAC:CONNECTORS_1X05_LOCK -> PCM2707:CONNECTORS_1X05_LOCK
- LED1, LED2: footprint PCM2707_DAC:LED_LED-0603 -> PCM2707:LED_LED-0603
- OUTPUT1: footprint PCM2707_DAC:CON-LSTB_MA03-1 -> PCM2707:CON-LSTB_MA03-1
- Q1: footprint PCM2707_DAC:CRYSTAL_HC49U-V -> PCM2707:CRYSTAL_HC49U-V
- SV1: footprint PCM2707_DAC:CON-LSTB_MA04-1 -> PCM2707:CON-LSTB_MA04-1
- U1: footprint PCM2707_DAC:PCM2707C -> PCM2707:PCM2707C
Changed lines of the file:
@@
 EESchema Schematic File Version 2
-LIBS:PCM2707_DAC
+LIBS:PCM2707
 LIBS:PCM2707_DAC-cache
 EELAYER 25 0
@@
 F 0 "C1" H 1510 4315 70  0000 L BNN
 F 1 "1uF" H 1509 4115 70  0000 L BNN
-F 2 "PCM2707_DAC:PASSIVES_0805" H 1440 3990 65  0001 L TNN
+F 2 "PCM2707:PASSIVES_0805" H 1440 3990 65  0001 L TNN
 F 3 "" H 1450 4200 60  0001 C CNN
 	1    1450 4200
@@
 F 0 "C2" H 2190 3425 70  0000 L BNN
 F 1 "10uF" H 2190 3235 70  0000 L BNN
-F 2 "PCM2707_DAC:PASSIVES_PANASONIC_C" H 2140 3190 65  0001 L TNN
+F 2 "PCM2707:PASSIVES_PANASONIC_C" H 2140 3190 65  0001 L TNN
 F 3 "" H 2150 3400 60  0001 C CNN
 	1    2150 3400
@@
 F 0 "C3" H 3310 3215 70  0000 L BNN
 F 1 "1uF" H 3310 3015 70  0000 L BNN
-F 2 "PCM2707_DAC:PASSIVES_0805" H 3240 2890 65  0001 L TNN
+F 2 "PCM2707:PASSIVES_0805" H 3240 2890 65  0001 L TNN
 F 3 "" H 3250 3100 60  0001 C CNN
 	1    3250 3100
@@
 F 0 "C4" H 3510 7215 70  0000 L BNN
 F 1 "22pF" H 3509 7015 70  0000 L BNN
-F 2 "PCM2707_DAC:PASSIVES_0805" H 3440 6890 65  0001 L TNN
+F 2 "PCM2707:PASSIVES_0805" H 3440 6890 65  0001 L TNN
 F 3 "" H 3450 7100 60  0001 C CNN
 	1    3450 7100
@@
 F 0 "C5" H 3910 7215 70  0000 L BNN
 F 1 "22pF" H 3909 7015 70  0000 L BNN
-F 2 "PCM2707_DAC:PASSIVES_0805" H 3840 6890 65  0001 L TNN
+F 2 "PCM2707:PASSIVES_0805" H 3840 6890 65  0001 L TNN
 F 3 "" H 3850 7100 60  0001 C CNN
 	1    3850 7100
@@
 F 0 "C6" H 4110 1915 70  0000 L BNN
 F 1 "22nF" H 4109 1715 70  0000 L BNN
-F 2 "PCM2707_DAC:PASSIVES_0805" H 4040 1590 65  0001 L TNN
+F 2 "PCM2707:PASSIVES_0805" H 4040 1590 65  0001 L TNN
 F 3 "" H 4050 1800 60  0001 C CNN
 	1    4050 1800
@@
 F 0 "C7" H 4210 3215 70  0000 L BNN
 F 1 "1uF" H 4210 3015 70  0000 L BNN
-F 2 "PCM2707_DAC:PASSIVES_0805" H 4140 2890 65  0001 L TNN
+F 2 "PCM2707:PASSIVES_0805" H 4140 2890 65  0001 L TNN
 F 3 "" H 4150 3100 60  0001 C CNN
 	1    4150 3100
@@
 F 0 "C8" H 4510 1915 70  0000 L BNN
 F 1 "22nF" H 4509 1715 70  0000 L BNN
-F 2 "PCM2707_DAC:PASSIVES_0805" H 4440 1590 65  0001 L TNN
+F 2 "PCM2707:PASSIVES_0805" H 4440 1590 65  0001 L TNN
 F 3 "" H 4450 1800 60  0001 C CNN
 	1    4450 1800
@@
 F 0 "C9" H 5410 5315 70  0000 L BNN
 F 1 "1uF" H 5409 5115 70  0000 L BNN
-F 2 "PCM2707_DAC:PASSIVES_0805" H 5340 4990 65  0001 L TNN
+F 2 "PCM2707:PASSIVES_0805" H 5340 4990 65  0001 L TNN
 F 3 "" H 5350 5200 60  0001 C CNN
 	1    5350 5200
@@
 F 0 "C10" H 5690 1025 70  0000 L BNN
 F 1 "100uF" H 5690 835 70  0000 L BNN
-F 2 "PCM2707_DAC:PASSIVES_PANASONIC_D" H 5640 790 65  0001 L TNN
+F 2 "PCM2707:PASSIVES_PANASONIC_D" H 5640 790 65  0001 L TNN
 F 3 "" H 5650 1000 60  0001 C CNN
 	1    5650 1000
@@
 F 0 "C11" H 5690 1425 70  0000 L BNN
 F 1 "100uF" H 5690 1235 70  0000 L BNN
-F 2 "PCM2707_DAC:PASSIVES_PANASONIC_D" H 5640 1190 65  0001 L TNN
+F 2 "PCM2707:PASSIVES_PANASONIC_D" H 5640 1190 65  0001 L TNN
 F 3 "" H 5650 1400 60  0001 C CNN
 	1    5650 1400
@@
 F 0 "C12" H 6710 5215 70  0000 L BNN
 F 1 "1uF" H 6709 5015 70  0000 L BNN
-F 2 "PCM2707_DAC:PASSIVES_0805" H 6640 4890 65  0001 L TNN
+F 2 "PCM2707:PASSIVES_0805" H 6640 4890 65  0001 L TNN
 F 3 "" H 6650 5100 60  0001 C CNN
 	1    6650 5100
@@
 F 0 "CON1" H 8450 2100 50  0000 L BNN
 F 1 "GND_CONNECTORSMD" H 8450 1701 50  0000 L BNN
-F 2 "PCM2707_DAC:GND_CONNECTOR" H 8840 1690 65  0001 L TNN
+F 2 "PCM2707:GND_CONNECTOR" H 8840 1690 65  0001 L TNN
 F 3 "" H 8850 1900 60  0001 C CNN
 	1    8850 1900
@@
 F 0 "DOUT1" H 5950 5570 60  0000 L BNN
 F 1 "87758-0216" H 5821 5655 70  0000 L BNN
-F 2 "PCM2707_DAC:CON-MOLEX_87758-0216" H 5821 5655 70  0001 L BNN
+F 2 "PCM2707:CON-MOLEX_87758-0216" H 5821 5655 70  0001 L BNN
 F 3 "" H 5850 5600 60  0001 C CNN
 	1    5850 5600
@@
 F 0 "DOUT1" H 5950 5770 60  0000 L BNN
 F 1 "87758-0216" H 5821 5855 70  0000 L BNN
-F 2 "PCM2707_DAC:CON-MOLEX_87758-0216" H 5821 5855 70  0001 L BNN
+F 2 "PCM2707:CON-MOLEX_87758-0216" H 5821 5855 70  0001 L BNN
 F 3 "" H 5850 5800 60  0001 C CNN
 	2    5850 5800
@@
 F 0 "J1" H 9650 4900 45  0000 L BNN
 F 1 "USB" H 9650 3800 45  0000 L BNN
-F 2 "PCM2707_DAC:MOLEX-47346-0001_MOLEX_47346-0001" H 9880 4550 20  0001 C CNN
+F 2 "PCM2707:MOLEX-47346-0001_MOLEX_47346-0001" H 9880 4550 20  0001 C CNN
 F 3 "" H 9850 4400 60  0001 C CNN
 	1    9850 4400
@@
 F 0 "JACK-OUT1" H 7150 1250 70  0000 L BNN
 F 1 "STEREOJACK" H 7150 700 70  0000 L BNN
-F 2 "PCM2707_DAC:STX3100" H 7440 890 65  0001 L TNN
+F 2 "PCM2707:STX3100" H 7440 890 65  0001 L TNN
 F 3 "" H 7450 1100 60  0001 C CNN
 	1    7450 1100
@@
 F 0 "JP1" H 951 5830 70  0000 L BNN
 F 1 "~" H 1040 5390 65  0001 L TNN
-F 2 "PCM2707_DAC:CONNECTORS_1X05_LOCK" H 1040 5290 65  0001 L TNN
+F 2 "PCM2707:CONNECTORS_1X05_LOCK" H 1040 5290 65  0001 L TNN
 F 3 "" H 1050 5500 60  0001 C CNN
 	1    1050 5500
@@
 F 0 "L1" H 7150 4400 70  0000 L BNN
 F 1 "1A FB" H 7150 4000 70  0000 L BNN
-F 2 "PCM2707_DAC:PASSIVES_0805" H 7040 3990 65  0001 L TNN
+F 2 "PCM2707:PASSIVES_0805" H 7040 3990 65  0001 L TNN
 F 3 "" H 7050 4200 60  0001 C CNN
 	1    7050 4200
@@
 F 0 "LED1" V 8590 2620 70  0000 L BNN
 F 1 "Blue" V 8675 2620 70  0000 L BNN
-F 2 "PCM2707_DAC:LED_LED-0603" H 8440 2590 65  0001 L TNN
+F 2 "PCM2707:LED_LED-0603" H 8440 2590 65  0001 L TNN
 F 3 "" H 8450 2800 60  0001 C CNN
 	1    8450 2800
@@
 F 0 "LED2" V 9190 2620 70  0000 L BNN
 F 1 "Blue" V 9275 2620 70  0000 L BNN
-F 2 "PCM2707_DAC:LED_LED-0603" H 9040 2590 65  0001 L TNN
+F 2 "PCM2707:LED_LED-0603" H 9040 2590 65  0001 L TNN
 F 3 "" H 9050 2800 60  0001 C CNN
 	1    9050 2800
@@
 F 0 "OUTPUT1" H 901 1530 70  0000 L BNN
 F 1 "AUDIO" H 900 1000 70  0000 L BNN
-F 2 "PCM2707_DAC:CON-LSTB_MA03-1" H 940 1090 65  0001 L TNN
+F 2 "PCM2707:CON-LSTB_MA03-1" H 940 1090 65  0001 L TNN
 F 3 "" H 950 1300 60  0001 C CNN
 	1    950  1300
@@
 F 0 "Q1" H 3750 6739 70  0000 L BNN
 F 1 "12MHz" H 3750 6600 70  0000 L BNN
-F 2 "PCM2707_DAC:CRYSTAL_HC49U-V" H 3640 6490 65  0001 L TNN
+F 2 "PCM2707:CRYSTAL_HC49U-V" H 3640 6490 65  0001 L TNN
 F 3 "" H 3650 6700 60  0001 C CNN
 	1    3650 6700
@@
 F 0 "R1" H 3500 6459 70  0000 L BNN
 F 1 "1MOhm" H 3500 6270 70  0000 L BNN
-F 2 "PCM2707_DAC:PASSIVES_0805" H 3640 6190 65  0001 L TNN
+F 2 "PCM2707:PASSIVES_0805" H 3640 6190 65  0001 L TNN
 F 3 "" H 3650 6400 60  0001 C CNN
 	1    3650 6400
@@
 F 0 "R2" H 3900 2159 70  0000 L BNN
 F 1 "16Ohm" H 3900 1970 70  0000 L BNN
-F 2 "PCM2707_DAC:PASSIVES_0805" H 4040 1890 65  0001 L TNN
+F 2 "PCM2707:PASSIVES_0805" H 4040 1890 65  0001 L TNN
 F 3 "" H 4050 2100 60  0001 C CNN
 	1    4050 2100
@@
 F 0 "R3" H 4000 6559 70  0000 L BNN
 F 1 "1.5kOhm" H 4000 6370 70  0000 L BNN
-F 2 "PCM2707_DAC:PASSIVES_0805" H 4140 6290 65  0001 L TNN
+F 2 "PCM2707:PASSIVES_0805" H 4140 6290 65  0001 L TNN
 F 3 "" H 4150 6500 60  0001 C CNN
 	1    4150 6500
@@
 F 0 "R4" H 4300 2159 70  0000 L BNN
 F 1 "16Ohm" H 4300 1970 70  0000 L BNN
-F 2 "PCM2707_DAC:PASSIVES_0805" H 4440 1890 65  0001 L TNN
+F 2 "PCM2707:PASSIVES_0805" H 4440 1890 65  0001 L TNN
 F 3 "" H 4450 2100 60  0001 C CNN
 	1    4450 2100
@@
 F 0 "R5" H 4800 1859 70  0000 L BNN
 F 1 "3.3kOhm" H 4800 1670 70  0000 L BNN
-F 2 "PCM2707_DAC:PASSIVES_0805" H 4940 1590 65  0001 L TNN
+F 2 "PCM2707:PASSIVES_0805" H 4940 1590 65  0001 L TNN
 F 3 "" H 4950 1800 60  0001 C CNN
 	1    4950 1800
@@
 F 0 "R6" H 5100 1859 70  0000 L BNN
 F 1 "3.3kOhm" H 5100 1670 70  0000 L BNN
-F 2 "PCM2707_DAC:PASSIVES_0805" H 5240 1590 65  0001 L TNN
+F 2 "PCM2707:PASSIVES_0805" H 5240 1590 65  0001 L TNN
 F 3 "" H 5250 1800 60  0001 C CNN
 	1    5250 1800
@@
 F 0 "R7" H 5800 4659 70  0000 L BNN
 F 1 "22Ohm" H 5800 4470 70  0000 L BNN
-F 2 "PCM2707_DAC:PASSIVES_0805" H 5940 4390 65  0001 L TNN
+F 2 "PCM2707:PASSIVES_0805" H 5940 4390 65  0001 L TNN
 F 3 "" H 5950 4600 60  0001 C CNN
 	1    5950 4600
@@
 F 0 "R8" H 5900 1859 70  0000 L BNN
 F 1 "3.3kOhm" H 5900 1670 70  0000 L BNN
-F 2 "PCM2707_DAC:PASSIVES_0805" H 6040 1590 65  0001 L TNN
+F 2 "PCM2707:PASSIVES_0805" H 6040 1590 65  0001 L TNN
 F 3 "" H 6050 1800 60  0001 C CNN
 	1    6050 1800
@@
 F 0 "R9" H 6100 4459 70  0000 L BNN
 F 1 "22Ohm" H 6100 4270 70  0000 L BNN
-F 2 "PCM2707_DAC:PASSIVES_0805" H 6240 4190 65  0001 L TNN
+F 2 "PCM2707:PASSIVES_0805" H 6240 4190 65  0001 L TNN
 F 3 "" H 6250 4400 60  0001 C CNN
 	1    6250 4400
@@
 F 0 "R10" H 6200 1859 70  0000 L BNN
 F 1 "3.3kOhm" H 6200 1670 70  0000 L BNN
-F 2 "PCM2707_DAC:PASSIVES_0805" H 6340 1590 65  0001 L TNN
+F 2 "PCM2707:PASSIVES_0805" H 6340 1590 65  0001 L TNN
 F 3 "" H 6350 1800 60  0001 C CNN
 	1    6350 1800
@@
 F 0 "R11" H 6400 3859 70  0000 L BNN
 F 1 "1.5kOhm" H 6400 3670 70  0000 L BNN
-F 2 "PCM2707_DAC:PASSIVES_0805" H 6540 3590 65  0001 L TNN
+F 2 "PCM2707:PASSIVES_0805" H 6540 3590 65  0001 L TNN
 F 3 "" H 6550 3800 60  0001 C CNN
 	1    6550 3800
@@
 F 0 "R12" H 8300 3359 70  0000 L BNN
 F 1 "560Ohm" H 8300 3170 70  0000 L BNN
-F 2 "PCM2707_DAC:PASSIVES_0805" H 8440 3090 65  0001 L TNN
+F 2 "PCM2707:PASSIVES_0805" H 8440 3090 65  0001 L TNN
 F 3 "" H 8450 3300 60  0001 C CNN
 	1    8450 3300
@@
 F 0 "R13" H 8900 3359 70  0000 L BNN
 F 1 "330Ohm" H 8900 3170 70  0000 L BNN
-F 2 "PCM2707_DAC:PASSIVES_0805" H 9040 3090 65  0001 L TNN
+F 2 "PCM2707:PASSIVES_0805" H 9040 3090 65  0001 L TNN
 F 3 "" H 9050 3300 60  0001 C CNN
 	1    9050 3300
@@
 F 0 "SV1" H 8500 5430 70  0000 L BNN
 F 1 "USB-WIRE" H 8501 4800 70  0000 L BNN
-F 2 "PCM2707_DAC:CON-LSTB_MA04-1" H 8540 4990 65  0001 L TNN
+F 2 "PCM2707:CON-LSTB_MA04-1" H 8540 4990 65  0001 L TNN
 F 3 "" H 8550 5200 60  0001 C CNN
 	1    8550 5200
@@
 F 0 "U1" H 3150 5000 45  0000 L BNN
 F 1 "PCM2707C" H 3150 4700 45  0000 L BNN
-F 2 "PCM2707_DAC:PCM2707C" H 3680 5050 20  0001 C CNN
+F 2 "PCM2707:PCM2707C" H 3680 5050 20  0001 C CNN
 F 3 "" H 3650 4900 60  0000 C CNN
 	1    3650 4900
